Commit message: Split ros2_control into separate j0 stepper and servo hardware blocks; add mock_hardware arg
- scara_arm_ros2_control.xacro: split single ros2_control block into _j0 (stepper via
  stepper_ros2_driver) and _servos (all Feetech joints via feetech_ros2_driver) blocks;
  add use_mock_hardware xacro arg; add velocity state interfaces and servo params (id,
  offset, gear_ratio, direction)
- Add config/scara_controllers.yaml
- urdf/mantis_gripper.xacro: minor fixes
- package.xml: add dependencies

Co-Authored-By: Claude Sonnet 4.6 <noreply@anthropic.com>

File: urdf/mantis_gripper.xacro (robot description, xacro)
@@ -2,5 +2,5 @@
 <robot xmlns:xacro="http://ros.org/wiki/xacro">
   <xacro:property name="M_SCALE" value="0.001"/>
-  <xacro:include filename="$(find scara_arm)/urdf/hardware.xacro" />
+  <xacro:include filename="$(find omni_bot2)/urdf/hardware.xacro" />
     <!-- side reflect parent -->
   <xacro:macro name="gripper_macro" params="parent">
@@ -24,5 +24,5 @@
    <visual>
       <geometry>
-        <mesh filename="package://scara_arm/mesh/claw_3_rr.stl" scale="${M_SCALE} ${M_SCALE} ${M_SCALE}"/>
+        <mesh filename="package://omni_bot2/mesh/claw_3_rr.stl" scale="${M_SCALE} ${M_SCALE} ${M_SCALE}"/>
       </geometry>
          <xacro:White/>
@@ -32,5 +32,5 @@
         <origin xyz="0 0 0" rpy="0 0 0" />
         <geometry>
-          <mesh filename="package://scara_arm/mesh/claw_3_rr.stl" scale="${M_SCALE} ${M_SCALE} ${M_SCALE}"/>
+          <mesh filename="package://omni_bot2/mesh/claw_3_rr.stl" scale="${M_SCALE} ${M_SCALE} ${M_SCALE}"/>
           </geometry>
       </collision>
@@ -48,5 +48,5 @@
    <visual>
       <geometry>
-        <mesh filename="package://scara_arm/mesh/claw_3_l.stl" scale="${M_SCALE} ${M_SCALE} ${M_SCALE}"/>
+        <mesh filename="package://omni_bot2/mesh/claw_3_l.stl" scale="${M_SCALE} ${M_SCALE} ${M_SCALE}"/>
       </geometry>
          <xacro:White/>
@@ -56,5 +56,5 @@
         <origin xyz="0 0 0" rpy="0 0 0" />
         <geometry>
-          <mesh filename="package://scara_arm/mesh/claw_3_l.stl" scale="${M_SCALE} ${M_SCALE} ${M_SCALE}"/>
+          <mesh filename="package://omni_bot2/mesh/claw_3_l.stl" scale="${M_SCALE} ${M_SCALE} ${M_SCALE}"/>
           </geometry>
       </collision>

File: urdf/scara_arm_ros2_control.xacro (robot description, xacro)
@@ -1,8 +1,16 @@
 <?xml version="1.0"?>
 <robot xmlns:xacro="http://www.ros.org/wiki/xacro">
+  <xacro:arg name="use_mock_hardware" default="false"/>
   <xacro:macro name="scara_arm_ros2_control" params="name">
-    <ros2_control name="${name}" type="system">
+    <!-- ── j0: prismatic lift — ESP32 + TMC2208 stepper on /dev/stepper ─────── -->
+    <ros2_control name="${name}_j0" type="system">
       <hardware>
-        <plugin>mock_components/GenericSystem</plugin>
+        <xacro:if value="$(arg use_mock_hardware)">
+          <plugin>mock_components/GenericSystem</plugin>
+        </xacro:if>
+        <xacro:unless value="$(arg use_mock_hardware)">
+          <plugin>stepper_ros2_driver/StepperHardwareInterface</plugin>
+          <param name="serial_port">/dev/stepper</param>
+        </xacro:unless>
       </hardware>
       <joint name="j0">
@@ -11,34 +19,112 @@
           <param name="initial_value">0.0</param>
         </state_interface>
+        <state_interface name="velocity">
+          <param name="initial_value">0.0</param>
+        </state_interface>
       </joint>
+    </ros2_control>
+    <!-- ── All Feetech servos (arm + head) on /dev/st_servo ─────────────────── -->
+    <!--  Single hardware block — LibSerial locks the port exclusively so only   -->
+    <!--  one FeetechHardwareInterface instance can own /dev/st_servo.           -->
+    <ros2_control name="${name}_servos" type="system">
+      <hardware>
+        <xacro:if value="$(arg use_mock_hardware)">
+          <plugin>mock_components/GenericSystem</plugin>
+        </xacro:if>
+        <xacro:unless value="$(arg use_mock_hardware)">
+          <plugin>feetech_ros2_driver/FeetechHardwareInterface</plugin>
+          <param name="usb_port">/dev/st_servo</param>
+        </xacro:unless>
+      </hardware>
+      <!-- Arm joints -->
       <joint name="j1">
+        <param name="id">9</param>
+        <param name="offset">2048</param>
+        <param name="gear_ratio">2.0</param>
+        <param name="direction">1</param>
         <command_interface name="position"/>
         <state_interface name="position">
           <param name="initial_value">0.0</param>
         </state_interface>
+        <state_interface name="velocity">
+          <param name="initial_value">0.0</param>
+        </state_interface>
       </joint>
       <joint name="j2">
+        <param name="id">8</param>
+        <param name="offset">2048</param>
+        <param name="gear_ratio">2.0</param>
+        <param name="direction">1</param>
         <command_interface name="position"/>
         <state_interface name="position">
           <param name="initial_value">0.0</param>
         </state_interface>
+        <state_interface name="velocity">
+          <param name="initial_value">0.0</param>
+        </state_interface>
       </joint>
       <joint name="j3">
+        <param name="id">19</param>
+        <param name="offset">2048</param>
+        <param name="gear_ratio">1.0</param>
+        <param name="direction">1</param>
         <command_interface name="position"/>
         <state_interface name="position">
           <param name="initial_value">0.0</param>
         </state_interface>
+        <state_interface name="velocity">
+          <param name="initial_value">0.0</param>
+        </state_interface>
       </joint>
       <joint name="j4">
+        <param name="id">17</param>
+        <param name="offset">2048</param>
+        <param name="gear_ratio">1.0</param>
+        <param name="direction">1</param>
         <command_interface name="position"/>
         <state_interface name="position">
           <param name="initial_value">0.0</param>
         </state_interface>
+        <state_interface name="velocity">
+          <param name="initial_value">0.0</param>
+        </state_interface>
       </joint>
       <joint name="gripper">
+        <param name="id">18</param>
+        <param name="offset">2048</param>
+        <param name="gear_ratio">1.0</param>
+        <param name="direction">1</param>
         <command_interface name="position"/>
         <state_interface name="position">
+          <param name="initial_value">-1.3</param>
+        </state_interface>
+        <state_interface name="velocity">
           <param name="initial_value">0.0</param>
         </state_interface>
+      </joint>
+      <!-- Head joints -->
+      <joint name="head_pan_joint">
+        <param name="initial_position">0.0</param>
+        <param name="id">4</param>
+        <param name="p_cofficient">20</param>
+        <param name="offset">2048</param>
+        <param name="gear_ratio">2.0</param>
+        <param name="direction">-1</param>
+        <param name="speed">3000</param>
+        <param name="acceleration">80</param>
+        <command_interface name="position"/>
+        <state_interface name="position"/>
+        <state_interface name="velocity"/>
+      </joint>
+      <joint name="head_tilt_joint">
+        <param name="initial_position">0.0</param>
+        <param name="id">5</param>
+        <param name="p_cofficient">20</param>
+        <param name="offset">2048</param>
+        <param name="gear_ratio">2.0</param>
+        <param name="direction">-1</param>
+        <command_interface name="position"/>
+        <state_interface name="position"/>
+        <state_interface name="velocity"/>
       </joint>
     </ros2_control>

Commit message: Add effort state interfaces to all joints; tune SCARA geometry and limits
- Add effort state_interface (initial 0.0) to j0–j4, gripper, head_pan,
  head_tilt so joint_states publishes 0.0 instead of NaN
- Fix j3 direction: 1 → -1
- Fix j2 offset: 2048 → 2100
- Tighten j1/j2 joint limits: ±2.356 → ±1.57 rad
- Adjust torso_link height 1.25 → 0.67, b2 width 0.18 → 0.12
- Move j4 origin x: 0.01 → 0.07
- Replace stale comment with xml declaration in mantis_gripper.xacro

Co-Authored-By: Claude Sonnet 4.6 <noreply@anthropic.com>

File: urdf/mantis_gripper.xacro (robot description, xacro)
@@ -1,3 +1,3 @@
-<!-- vis_lecture/xacro/basic5_h.xacro -->
+<?xml version="1.0"?>
 <robot xmlns:xacro="http://ros.org/wiki/xacro">
   <xacro:property name="M_SCALE" value="0.001"/>

File: urdf/robbie_scara.urdf.xacro (robot description, xacro)
@@ -75,5 +75,5 @@
   <link name="oak"/>
   <!-- === Torso ==================================================================== -->
-  <xacro:my_box name="torso_link" lwh="0.03 0.15 1.25" xyz="0 0 0" rpy="0 0 0" mass="0.1" material="Gazebo/FlatBlack">
+  <xacro:my_box name="torso_link" lwh="0.03 0.15 0.67" xyz="0 0 0" rpy="0 0 0" mass="0.1" material="Gazebo/FlatBlack">
 	        <xacro:grey2 />
         </xacro:my_box>
@@ -90,5 +90,5 @@
 	        <xacro:grey2 />
         </xacro:my_cylinder>
-<xacro:my_box name="b2" lwh="0.18 0.065 0.03" xyz="0 0 0" rpy="0 0 0" mass="0.1" material="Gazebo/FlatBlack">
+<xacro:my_box name="b2" lwh="0.12 0.065 0.03" xyz="0 0 0" rpy="0 0 0" mass="0.1" material="Gazebo/FlatBlack">
 	        <xacro:grey2 />
         </xacro:my_box>
@@ -188,5 +188,5 @@
         <axis xyz="0 0 1"/>
     	<origin xyz="0.045 0 0.05 " rpy="0 0 0" />
-        <limit effort="1000.0" lower="-2.356" upper="2.356" velocity="0.5"/>
+        <limit effort="1000.0" lower="-1.57" upper="1.57" velocity="0.5"/>
 </joint>
 <joint name="b1" type="fixed">
@@ -200,5 +200,5 @@
         <axis xyz="0 0 1"/>
     	<origin xyz="0.045 0 -0.05 " rpy="0 0 0" />
-        <limit effort="1000.0" lower="-2.356" upper="2.356" velocity="0.5"/>
+        <limit effort="1000.0" lower="-1.57" upper="1.57" velocity="0.5"/>
 </joint>
 <joint name="b2" type="fixed">
@@ -218,5 +218,5 @@
     	<child link="j4" />
         <axis xyz="0 1 0"/>
-    	<origin xyz="0.01 0 -0.02 " rpy="0 0 0" />
+    	<origin xyz="0.07 0 -0.02 " rpy="0 0 0" />
         <limit effort="1000.0" lower="-1.57" upper="1.57" velocity="0.5"/>
 </joint>

File: urdf/scara_arm_ros2_control.xacro (robot description, xacro)
@@ -20,4 +20,7 @@
         </state_interface>
         <state_interface name="velocity">
+          <param name="initial_value">0.0</param>
+        </state_interface>
+        <state_interface name="effort">
           <param name="initial_value">0.0</param>
         </state_interface>
@@ -50,8 +53,11 @@
           <param name="initial_value">0.0</param>
         </state_interface>
+        <state_interface name="effort">
+          <param name="initial_value">0.0</param>
+        </state_interface>
       </joint>
       <joint name="j2">
         <param name="id">8</param>
-        <param name="offset">2048</param>
+        <param name="offset">2100</param>
         <param name="gear_ratio">2.0</param>
         <param name="direction">1</param>
@@ -63,4 +69,7 @@
           <param name="initial_value">0.0</param>
         </state_interface>
+        <state_interface name="effort">
+          <param name="initial_value">0.0</param>
+        </state_interface>
       </joint>
       <joint name="j3">
@@ -68,5 +77,5 @@
         <param name="offset">2048</param>
         <param name="gear_ratio">1.0</param>
-        <param name="direction">1</param>
+        <param name="direction">-1</param>
         <command_interface name="position"/>
         <state_interface name="position">
@@ -74,4 +83,7 @@
         </state_interface>
         <state_interface name="velocity">
+          <param name="initial_value">0.0</param>
+        </state_interface>
+        <state_interface name="effort">
           <param name="initial_value">0.0</param>
         </state_interface>
@@ -89,4 +101,7 @@
           <param name="initial_value">0.0</param>
         </state_interface>
+        <state_interface name="effort">
+          <param name="initial_value">0.0</param>
+        </state_interface>
       </joint>
       <joint name="gripper">
@@ -100,4 +115,7 @@
         </state_interface>
         <state_interface name="velocity">
+          <param name="initial_value">0.0</param>
+        </state_interface>
+        <state_interface name="effort">
           <param name="initial_value">0.0</param>
         </state_interface>
@@ -116,4 +134,5 @@
         <state_interface name="position"/>
         <state_interface name="velocity"/>
+        <state_interface name="effort"/>
       </joint>
       <joint name="head_tilt_joint">
@@ -127,4 +146,5 @@
         <state_interface name="position"/>
         <state_interface name="velocity"/>
+        <state_interface name="effort"/>
       </joint>
     </ros2_control>

Commit message: Clean up colour macro names in hardware.xacro; update all URDF call sites
Renamed macros to remove numbers and capitals:
  White        → white
  grey1        → light_grey
  grey2        → grey
  grey3        → pale_grey
  ax12_color   → dark_grey  (removed duplicate definition)
  bracket_color→ off_white
  cyan1/2/3    → cyan_light / cyan / cyan_dark
  yellow2      → removed (duplicate of yellow)
  green1       → green
  green2       → lime
  blue         → removed duplicate definition
  default_inertial → removed duplicate definition
  F3_bracket   → removed stale inline material block

Updated robbie.urdf.xacro, robbie_scara.urdf.xacro, mantis_gripper.xacro
to use new names throughout.

Co-Authored-By: Claude Sonnet 4.6 <noreply@anthropic.com>

File: urdf/mantis_gripper.xacro (robot description, xacro)
@@ -26,5 +26,5 @@
         <mesh filename="package://omni_bot2/mesh/claw_3_rr.stl" scale="${M_SCALE} ${M_SCALE} ${M_SCALE}"/>
       </geometry>
-         <xacro:White/>
+         <xacro:white/>
       <origin rpy="0 0 0" xyz="0 0 0"/>
     </visual>
@@ -50,5 +50,5 @@
         <mesh filename="package://omni_bot2/mesh/claw_3_l.stl" scale="${M_SCALE} ${M_SCALE} ${M_SCALE}"/>
       </geometry>
-         <xacro:White/>
+         <xacro:white/>
       <origin rpy="0 0 0" xyz="0 0 0"/>
     </visual>

File: urdf/robbie.urdf.xacro (robot description, xacro)
@@ -49,5 +49,5 @@
               scale="${M_SCALE} ${M_SCALE} ${M_SCALE}"/>
       </geometry>
-      <xacro:grey2/>
+      <xacro:grey/>
     </visual>
     <collision>
@@ -65,5 +65,5 @@
               scale="${M_SCALE} ${M_SCALE} ${M_SCALE}"/>
       </geometry>
-      <xacro:grey1/>
+      <xacro:light_grey/>
     </visual>
     <collision>

File: urdf/robbie_scara.urdf.xacro (robot description, xacro)
@@ -47,5 +47,5 @@
               scale="${M_SCALE} ${M_SCALE} ${M_SCALE}"/>
       </geometry>
-      <xacro:grey2/>
+      <xacro:grey/>
     </visual>
     <collision>
@@ -63,5 +63,5 @@
               scale="${M_SCALE} ${M_SCALE} ${M_SCALE}"/>
       </geometry>
-      <xacro:grey1/>
+      <xacro:light_grey/>
     </visual>
     <collision>
@@ -76,26 +76,26 @@
   <!-- === Torso ==================================================================== -->
   <xacro:my_box name="torso_link" lwh="0.03 0.15 0.67" xyz="0 0 0" rpy="0 0 0" mass="0.1" material="Gazebo/FlatBlack">
-	        <xacro:grey2 />
+	        <xacro:grey />
         </xacro:my_box>
 <xacro:my_box name="j0" lwh="0.15 0.075 0.04" xyz="0 0 0" rpy="0 0 0" mass="0.1" material="Gazebo/FlatBlack">
-	        <xacro:grey2 />
+	        <xacro:grey />
         </xacro:my_box>
 <xacro:my_cylinder name="j1" r="0.02" l ="0.04" xyz="0 0 0" rpy="0 0 0" mass="0.1" material="Gazebo/FlatBlack">
-	        <xacro:grey2 />
+	        <xacro:grey />
         </xacro:my_cylinder>
  <xacro:my_box name="b1" lwh="0.15 0.075 0.04" xyz="0 0 0" rpy="0 0 0" mass="0.1" material="Gazebo/FlatBlack">
-	        <xacro:grey2 />
+	        <xacro:grey />
         </xacro:my_box>
 <xacro:my_cylinder name="j2" r="0.02" l ="0.04" xyz="0 0 0" rpy="0 0 0" mass="0.1" material="Gazebo/FlatBlack">
-	        <xacro:grey2 />
+	        <xacro:grey />
         </xacro:my_cylinder>
 <xacro:my_box name="b2" lwh="0.12 0.065 0.03" xyz="0 0 0" rpy="0 0 0" mass="0.1" material="Gazebo/FlatBlack">
-	        <xacro:grey2 />
+	        <xacro:grey />
         </xacro:my_box>
 <xacro:my_cylinder name="j3" r="0.02" l ="0.02" xyz="0 0 0" rpy="0 0 0" mass="0.1" material="Gazebo/FlatBlack">
-	        <xacro:grey2 />
+	        <xacro:grey />
         </xacro:my_cylinder>
 <xacro:my_cylinder name="j4" r="0.02" l ="0.02" xyz="0 0 0" rpy="0 0 0" mass="0.1" material="Gazebo/FlatBlack">
-	        <xacro:yellow2 />
+	        <xacro:yellow />
         </xacro:my_cylinder>
   <joint name="base_footprint_joint" type="fixed">
@@ -123,5 +123,5 @@
     <parent link="torso_link"/>
     <child  link="head_pan"/>
-    <origin xyz="0 0 0.625" rpy="0 0 0"/>
+    <origin xyz="0 0 0.32" rpy="0 0 0"/>
     <axis   xyz="0 0 1"/>
     <limit lower="-${joint_limit}" upper="${joint_limit}" effort="1" velocity="1.0"/>
